File: Hardware/Big_Red_Box_Proto_Board.brd (EAGLE design)
At the start: 150 x 82 mm, 5 parts

Commit message: added creative commons license and engineer name
Parts:
- added E$6: (no value), SparkFun-Aesthetics:CREATIVE_COMMONS
Other:
- board text added: "Casey Kuhns"
Changed lines of the file:
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@@
 <setting verticaltext="up"/>
 </settings>
-<grid distance="0.01" unitdist="inch" unit="inch" style="lines" multiple="1" display="yes" altdistance="0.025" altunitdist="inch" altunit="inch"/>
+<grid distance="0.1" unitdist="inch" unit="inch" style="lines" multiple="1" display="yes" altdistance="0.025" altunitdist="inch" altunit="inch"/>
 <layers>
 <layer number="1" name="Top" color="4" fill="1" visible="yes" active="yes"/>
@@
 <wire x1="0.254" y1="34.036" x2="0.254" y2="-32.004" width="0.2032" layer="20"/>
 <wire x1="-0.254" y1="34.036" x2="-0.254" y2="-32.004" width="0.2032" layer="20"/>
+<text x="-45.72" y="-86.36" size="1.778" layer="51">Casey Kuhns</text>
 </plain>
 <attributes>
@@
 <element name="E$4" library="SparkFun-Aesthetics" package="OSHW-LOGO-S" value="" x="34.29" y="-31.75"/>
 <element name="E$5" library="SparkFun-Aesthetics" package="OSHW-LOGO-S" value="" x="40.64" y="-31.75" rot="MR0"/>
+<element name="E$6" library="SparkFun-Aesthetics" package="CREATIVE_COMMONS" value="" x="-73.66" y="-86.36"/>
 </elements>
 <signals>
